Commit message: single-line-lidar to multi-lines-lidar

File: src/patrolbot_description/urdf/body.xacro (robot description, xacro)
@@ -87,5 +87,6 @@
         <material name="warning_black"/>
       </visual>
-      <xacro:inertial_box mass="${mass_led_bezel}" x="0.020" y="0.160" z="0.400" xyz="0 0 0"/>
+      <xacro:inertial_box mass="${mass_led_bezel}"
+        x="0.020" y="0.160" z="0.400" xyz="0 0 0"/>
     </link>
     <joint name="led_screen_joint" type="fixed">
@@ -102,5 +103,6 @@
         <material name="led_red"/>
       </visual>
-      <xacro:inertial_box mass="${mass_led_screen}" x="0.008" y="0.150" z="0.360" xyz="0 0 0"/>
+      <xacro:inertial_box mass="${mass_led_screen}"
+        x="0.008" y="0.150" z="0.360" xyz="0 0 0"/>
     </link>
     <!-- ===================== red / blue strobes ===================== -->
@@ -122,5 +124,8 @@
           <material name="${material}"/>
         </visual>
-        <xacro:inertial_box mass="${mass_strobe}" x="0.050" y="0.040" z="0.020" xyz="0 0 0"/>
+        <xacro:inertial_box
+          mass="${mass_strobe}"
+          x="0.050" y="0.040" z="0.020"
+          xyz="0 0 0"/>
       </link>
     </xacro:macro>

File: src/patrolbot_description/urdf/chassis.xacro (robot description, xacro)
@@ -30,5 +30,7 @@
       </collision>
       <xacro:inertial_box mass="${mass_base}"
-                          x="${chassis_length}" y="${chassis_width}" z="${chassis_height}"
+                          x="${chassis_length}"
+                          y="${chassis_width}"
+                          z="${chassis_height}"
                           xyz="0 0 0"/>
     </link>
@@ -52,5 +54,7 @@
           <origin xyz="0 0 0" rpy="${pi/2} 0 0"/>
           <geometry>
-            <cylinder radius="${wheel_radius * 0.45}" length="${wheel_width + 0.004}"/>
+            <cylinder
+              radius="${wheel_radius * 0.45}"
+              length="${wheel_width + 0.004}"/>
           </geometry>
           <material name="aluminium"/>
@@ -59,5 +63,7 @@
           <origin xyz="0 0 0" rpy="${pi/2} 0 0"/>
           <geometry>
-            <cylinder radius="${wheel_radius}" length="${wheel_width}"/>
+            <cylinder
+              radius="${wheel_radius}"
+              length="${wheel_width}"/>
           </geometry>
         </collision>

File: src/patrolbot_description/urdf/mast_gimbal.xacro (robot description, xacro)
@@ -40,5 +40,6 @@
         <origin xyz="0 0 0" rpy="0 0 0"/>
         <axis xyz="0 0 1"/>
-        <limit lower="0.0" upper="${travel}" effort="200.0" velocity="0.20"/>
+        <limit lower="0.0" upper="${travel}"
+              effort="200.0" velocity="0.20"/>
         <dynamics damping="50.0" friction="25.0"/>
       </joint>
@@ -51,16 +52,21 @@
           <material name="aluminium"/>
         </visual>
-        <xacro:inertial_cylinder mass="${mass}" radius="${radius}" length="${mast_tube_length}"
-                                 xyz="0 0 ${-mast_tube_length/2.0}"/>
+        <xacro:inertial_cylinder mass="${mass}"
+              radius="${radius}"
+              length="${mast_tube_length}"
+              xyz="0 0 ${-mast_tube_length/2.0}"/>
       </link>
     </xacro:macro>
     <xacro:patrolbot_mast_stage index="1" parent="mast_base_link"
-                                radius="${mast_stage1_radius}" mass="${mass_mast_stage1}"
+                                radius="${mast_stage1_radius}"
+                                mass="${mass_mast_stage1}"
                                 travel="${mast_stage_travel}"/>
     <xacro:patrolbot_mast_stage index="2" parent="mast_stage1_link"
-                                radius="${mast_stage2_radius}" mass="${mass_mast_stage2}"
+                                radius="${mast_stage2_radius}"
+                                mass="${mass_mast_stage2}"
                                 travel="${mast_stage_travel}"/>
     <xacro:patrolbot_mast_stage index="3" parent="mast_stage2_link"
-                                radius="${mast_stage3_radius}" mass="${mass_mast_stage3}"
+                                radius="${mast_stage3_radius}"
+                                mass="${mass_mast_stage3}"
                                 travel="${mast_stage_travel}"/>
     <!-- ===================== three-axis gimbal ===================== -->
@@ -81,6 +87,7 @@
         <material name="aluminium"/>
       </visual>
-      <xacro:inertial_cylinder mass="${mass_gimbal_yaw}" radius="0.028" length="0.020"
-                               xyz="0 0 0.010"/>
+      <xacro:inertial_cylinder mass="${mass_gimbal_yaw}"
+        radius="0.028" length="0.020"
+        xyz="0 0 0.010"/>
     </link>
     <joint name="gimbal_pitch_joint" type="revolute">
@@ -100,6 +107,6 @@
         <material name="dark_grey"/>
       </visual>
-      <xacro:inertial_box mass="${mass_gimbal_pitch}" x="0.050" y="0.050" z="0.030"
-                          xyz="0 0 0.015"/>
+      <xacro:inertial_box mass="${mass_gimbal_pitch}"
+          x="0.050" y="0.050" z="0.030" xyz="0 0 0.015"/>
     </link>
     <joint name="gimbal_roll_joint" type="revolute">

File: src/patrolbot_description/urdf/patrolbot.urdf.xacro (robot description, xacro)
@@ -4,5 +4,5 @@
   Usage:
     xacro patrolbot.urdf.xacro > /tmp/patrolbot.urdf
-    xacro patrolbot.urdf.xacro lidar_samples:=360 controllers_file:=/abs/path.yaml
+    xacro patrolbot.urdf.xacro lidar_lines:=16 lidar_samples:=360 controllers_file:=/abs/path.yaml
   The model targets ROS 2 Jazzy + Gazebo Harmonic.  See README.md in this
   directory for the world plugins and bridge topics the simulation needs.
@@ -13,6 +13,17 @@
              default="$(find patrolbot_description)/config/ros2_control.yaml"/>
   <xacro:arg name="lidar_samples" default="720"/>
+  <xacro:arg name="lidar_lines" default="32"/>
   <xacro:arg name="lidar_max_range" default="100.0"/>
   <xacro:arg name="lidar_update_rate" default="10.0"/>
+  <!-- Multi-line lidar presets (placeholder values until the sensor is selected):
+         32 lines: vertical FOV -25 deg ... +15 deg
+         16 lines: vertical FOV -15 deg ... +15 deg
+       Only 16 and 32 are supported; any other value falls back to the
+       32-line preset.  The horizontal resolution is still controlled by
+       lidar_samples (points per ring). -->
+  <xacro:property name="lidar_line_count" value="$(arg lidar_lines)"/>
+  <xacro:property name="lidar_vertical_min_angle"
+                  value="${-0.2618 if int(lidar_line_count) == 16 else -0.4363}"/>
+  <xacro:property name="lidar_vertical_max_angle" value="0.2618"/>
   <xacro:arg name="imu_update_rate" default="100.0"/>
   <xacro:arg name="gnss_update_rate" default="10.0"/>

File: src/patrolbot_description/urdf/sensors.xacro (robot description, xacro)
@@ -1,6 +1,7 @@
 <?xml version="1.0"?>
 <!--
-  Sensor suite: 100 m lidar, IMU, RTK/GNSS, 1080p panorama camera,
-  gimbal camera (80 m violation capture) and the blind-spot sensor frames.
+  Sensor suite: 100 m multi-line lidar (32-line default, 16-line
+  selectable), IMU, RTK/GNSS, 1080p panorama camera, gimbal camera
+  (80 m violation capture) and the blind-spot sensor frames.
   Only the lidar / IMU / GNSS / cameras carry Gazebo sensors.  The mmWave
   radar and the six ultrasonic sensors are modelled as frames + visuals;
@@ -11,14 +12,20 @@
 <robot xmlns:xacro="http://www.ros.org/wiki/xacro">
   <xacro:macro name="patrolbot_sensors">
-    <!-- ===================== 100 m 2D lidar ===================== -->
-    <!-- Mounted at the front of the cone top; the scan plane is 0.882 m
-         above the ground.  Everything forward of and beside the lidar is
-         kept below that plane while the mast is collapsed (strobes and
-         mast collar top out at 0.875 m, panorama camera at 0.793 m), so the
-         forward and side sectors are unobstructed.  The gimbal head crosses
-         the plane while the mast is collapsed and blanks about +-21 deg
-         around the rear; intermediate lift states stay within that, and with
-         the mast extended the stage-1 tube is the only occluder, narrowing
-         the blanking to about +-18 deg.  See README.md. -->
+    <!-- ===================== 100 m multi-line lidar ===================== -->
+    <!-- Mounted at the front of the cone top; the scan origin is 0.882 m
+         above the ground.  Default is 32 lines, switchable to 16 lines:
+           lidar_lines:=32  -> vertical FOV -25 deg ... +15 deg
+           lidar_lines:=16  -> vertical FOV -15 deg ... +15 deg
+         These FOVs are placeholders until the actual sensor is selected;
+         they only cover the common mechanical 16/32-line families.
+         With a vertical FOV the lidar also sees the ground and the nearby
+         cone top.  Returns closer than range.min (0.20 m) are discarded,
+         so the body/ground immediately around the lidar is self-filtered;
+         ground points beyond 1.9-3.3 m (depending on the lower FOV) are
+         intentional and useful for ground segmentation.  The rear gimbal
+         head still blanks the low beams around the rear (about +-21 deg
+         on the horizontal plane when the mast is collapsed); re-check the
+         exact 3D self-occlusion against the selected sensor.  See
+         README.md. -->
     <joint name="lidar_joint" type="fixed">
       <parent link="body_link"/>
@@ -35,5 +42,5 @@
         <material name="aluminium"/>
       </visual>
-      <!-- base plate, just above the scan plane -->
+      <!-- base plate, just above the scan origin -->
       <visual>
         <origin xyz="0 0 0.003" rpy="0 0 0"/>
@@ -43,5 +50,6 @@
         <material name="warning_black"/>
       </visual>
-      <!-- low-profile housing -->
+      <!-- low-profile housing (placeholder; replace with the selected
+           16/32-line unit's diameter, height and mass) -->
       <visual>
         <origin xyz="0 0 0.017" rpy="0 0 0"/>
@@ -51,6 +59,8 @@
         <material name="dark_grey"/>
       </visual>
-      <!-- top cap; the lidar is 0.035 m tall so it stays out of the
-           gimbal camera's forward field of view in the collapsed pose -->
+      <!-- top cap; the housing is deliberately kept low so it stays out
+           of the gimbal camera's forward field of view in the collapsed
+           pose.  A physically larger 32-line unit may require raising the
+           camera or moving the lidar; this is a placeholder. -->
       <visual>
         <origin xyz="0 0 0.0315" rpy="0 0 0"/>
@@ -67,5 +77,5 @@
         <always_on>true</always_on>
         <update_rate>$(arg lidar_update_rate)</update_rate>
-        <visualize>false</visualize>
+        <visualize>true</visualize>
         <topic>/scan</topic>
         <gz_frame_id>lidar_link</gz_frame_id>
@@ -79,8 +89,8 @@
             </horizontal>
             <vertical>
-              <samples>1</samples>
+              <samples>$(arg lidar_lines)</samples>
               <resolution>1</resolution>
-              <min_angle>0</min_angle>
-              <max_angle>0</max_angle>
+              <min_angle>${lidar_vertical_min_angle}</min_angle>
+              <max_angle>${lidar_vertical_max_angle}</max_angle>
             </vertical>
           </scan>
@@ -322,5 +332,8 @@
         <material name="warning_black"/>
       </visual>
-      <xacro:inertial_box mass="${mass_mmwave}" x="0.025" y="0.100" z="0.050" xyz="0 0 0"/>
+      <xacro:inertial_box
+        mass="${mass_mmwave}"
+        x="0.025"  y="0.100" z="0.050"
+        xyz="0 0 0"/>
     </link>
     <!-- ===================== ultrasonic blind-spot sensors ===================== -->
@@ -339,14 +352,23 @@
           <material name="dark_grey"/>
         </visual>
-        <xacro:inertial_cylinder mass="${mass_ultrasonic}" radius="0.013" length="0.012"
-                                 xyz="0 0 0"/>
+        <xacro:inertial_cylinder
+          mass="${mass_ultrasonic}"
+          radius="0.013"
+          length="0.012"
+          xyz="0 0 0"/>
       </link>
     </xacro:macro>
-    <xacro:patrolbot_ultrasonic name="front_left"  x="0.214" y="0.100"  rpy="0 ${pi/2} 0"/>
-    <xacro:patrolbot_ultrasonic name="front_right" x="0.214" y="-0.100" rpy="0 ${pi/2} 0"/>
-    <xacro:patrolbot_ultrasonic name="rear_left"   x="-0.214" y="0.100"  rpy="0 ${pi/2} 0"/>
-    <xacro:patrolbot_ultrasonic name="rear_right"  x="-0.214" y="-0.100" rpy="0 ${pi/2} 0"/>
-    <xacro:patrolbot_ultrasonic name="left"        x="0.0" y="0.164"  rpy="${pi/2} 0 0"/>
-    <xacro:patrolbot_ultrasonic name="right"       x="0.0" y="-0.164" rpy="${pi/2} 0 0"/>
+    <xacro:patrolbot_ultrasonic name="front_left"
+      x="0.214" y="0.100"  rpy="0 ${pi/2} 0"/>
+    <xacro:patrolbot_ultrasonic name="front_right"
+      x="0.214" y="-0.100" rpy="0 ${pi/2} 0"/>
+    <xacro:patrolbot_ultrasonic name="rear_left"
+      x="-0.214" y="0.100"  rpy="0 ${pi/2} 0"/>
+    <xacro:patrolbot_ultrasonic name="rear_right"
+      x="-0.214"  y="-0.100"  rpy="0 ${pi/2} 0"/>
+    <xacro:patrolbot_ultrasonic name="left"
+      x="0.0" y="0.164"  rpy="${pi/2} 0 0"/>
+    <xacro:patrolbot_ultrasonic name="right"
+      x="0.0" y="-0.164" rpy="${pi/2} 0 0"/>
   </xacro:macro>
 </robot>
